File: 03_electrical/esp32_nodemcu/power.kicad_sch (KiCad schematic)
At the start: 0 parts

Commit message: KiCad save
Parts:
- added C0, C1, C2, C3, C4, C5, C6: 220 nF, symbol Device:C_US
- added C7: 100 nF, symbol Device:C_US
- added J10: Conn_01x02, Connector_AMASS:AMASS_XT60PW-F_1x02_P7.20mm_Horizontal, symbol Connector_Generic:Conn_01x02
- added J9: Conn_01x07_Pin, Connector_JST:JST_XH_B7B-XH-A_1x07_P2.50mm_Vertical, symbol Connector:Conn_01x07_Pin
- added R0, R1, R2, R3, R4, R5, R6: 20 Ω, symbol Device:R_US
- added R10: 1 mΩ, symbol Device:R_US
- added R11, R12: 100 Ω, symbol Device:R_US
- added R13: 5.1 kΩ, symbol Device:R_US
- added R7, R8: 4.7 k, symbol Device:R_US
- added R9: 10 k, symbol Device:R_US
- added U2: BQ76942PFBR, BQ76942PFBR:PFB0048A_N, symbol BQ76942PFBR:BQ76942PFBR
Connections:
- new net: R13.2, U2.45 (CHG)
- new net: J9.3 (Pin_3), R2.1
- new net: C2.1, C3.2, R2.2, U2.14 (VC2)
- new net: J9.2 (Pin_2), R1.1
- new net: J9.4 (Pin_4), R3.1
- new net: J9.5 (Pin_5), R4.1
- new net: J9.6 (Pin_6), R5.1
- new net: J9.7 (Pin_7), R6.1
- new net: C1.1, C2.2, R1.2, U2.15 (VC1)
- new net: C4.1, C5.2, R4.2, U2.12 (VC4)
- new net: C7.2, R12.1, U2.20 (SRN)
- new net: C3.1, C4.2, R3.2, U2.13 (VC3)
- new net: C0.1, R0.2, U2.16 (VC0)
- new net: C6.1, R6.2, U2.48 (VC10)
- new net: C5.1, C6.2, R5.2, U2.10 (VC5), U2.2 (VC9), U2.4 (VC8), U2.6 (VC7), U2.8 (VC6)
- new net: C7.1, R11.1, U2.18 (SRP)
- new net +3V3: R7.2, R8.2, R9.2
- new net +BATT: J10.1 (Pin_1)
- new net -BATT: J10.2 (Pin_2)
- new net BMS_INT: R9.1, U2.25 (ALERT)
- new net GND: R10.1, R12.2
- new net I2C_SCL: R7.1, U2.26 (SCL)
- new net I2C_SDA: R8.1, U2.27 (SDA)
- new net SHUNT_BAT: J9.1 (Pin_1), R0.1, R10.2, R11.2
- new net VSS: C0.2, C1.2, U2.17 (VSS), U2.22 (TS2), U2.33 (RST_SHUT), U2.36 (REGIN), U2.37 (BREG)
- no-connect marks 0 -> 13
Other:
- note added: "B6 B5 B4 B3 B2 B1 B0"
- note added: "BAT_P - Raw Battery Positive BAT_N - Raw Battery Negative"
- note added: "NC OR VSS"
- note added: "SHUNT"
- note added: "VBAT - Protected Battery Positive"
- note added: "VSS -- NTC --"
- note removed: "BQ25756"
- note removed: "BQ76942"
- note removed: "LT8609S"
- note removed: "TPS25751A 60 W max"
- note removed: "TPSM828302"
