File: 03_electrical/esp32_nodemcu/esp32_nodemcu.kicad_pcb (KiCad board)
At the start: 2 copper layers, 104.1 x 132.1 mm, 2 parts

Commit message: KiCad save
Parts:
- added A2: Adafruit_CAN_Pal_TJA1051T3, Adafruit_CAN_Pal_TJA1051T3:Adafruit_CAN_Pal_TJA1051T3, F.Cu at (182.3, 140.0)
- added A3: RadioMaster_RP2_V2, RadioMaster_RP2_V2:RadioMaster_RP2_V2, F.Cu at (175.8, 116.4)
- added C4: 10 pF, Capacitor_SMD:C_0603_1608Metric_Pad1.08x0.95mm_HandSolder, F.Cu at (121.6, 105.8)
- added C5: 22 μF, Capacitor_SMD:C_1206_3216Metric_Pad1.33x1.80mm_HandSolder, F.Cu at (114.8, 114.4)
- added C_IN1: 4.7 μF, Capacitor_SMD:C_1206_3216Metric_Pad1.33x1.80mm_HandSolder, F.Cu at (125.7, 113.2)
- added C_VCC1: 1 μF, Capacitor_SMD:C_0603_1608Metric_Pad1.08x0.95mm_HandSolder, F.Cu at (116.0, 110.6)
- added DS1: Waveshare_2inch_LCD_ST7789VW, Waveshare_2inch_LCD_ST7789VW:Waveshare_2inch_LCD_ST7789VW, F.Cu at (246.3, 108.1)
- added H1: MountingHole, MountingHole:MountingHole_3.5mm_Pad_TopBottom, F.Cu at (159.2, 96.9)
- added H2: MountingHole, MountingHole:MountingHole_3.5mm_Pad_TopBottom, F.Cu at (260.8, 96.9)
- added H3: MountingHole, MountingHole:MountingHole_3.5mm_Pad_TopBottom, F.Cu at (159.2, 173.1)
- added H4: MountingHole, MountingHole:MountingHole_3.5mm_Pad_TopBottom, F.Cu at (260.8, 173.1)
- added J1: CAN_Node_3Pin, Connector_PinHeader_2.54mm:PinHeader_1x03_P2.54mm_Vertical, F.Cu at (252.7, 126.8)
- added J10: Screw_Terminal_01x02, TerminalBlock_Phoenix:TerminalBlock_Phoenix_MKDS-1,5-2-5.08_1x02_P5.08mm_Horizontal, F.Cu at (283.1, 123.2)
- added J11: Screw_Terminal_01x02, TerminalBlock_Phoenix:TerminalBlock_Phoenix_MKDS-1,5-2-5.08_1x02_P5.08mm_Horizontal, F.Cu at (283.1, 135.4)
- added J2: CAN_Node_3Pin, Connector_PinHeader_2.54mm:PinHeader_1x03_P2.54mm_Vertical, F.Cu at (252.7, 136.9)
- added J3: CAN_Node_3Pin, Connector_PinHeader_2.54mm:PinHeader_1x03_P2.54mm_Vertical, F.Cu at (252.7, 147.1)
- added J4: CAN_Node_3Pin, Connector_PinHeader_2.54mm:PinHeader_1x03_P2.54mm_Vertical, F.Cu at (252.7, 157.2)
- added J5: Screw_Terminal_01x02, TerminalBlock_Phoenix:TerminalBlock_Phoenix_MKDS-1,5-2-5.08_1x02_P5.08mm_Horizontal, B.Cu at (240.2, 126.8)
- added J6: Screw_Terminal_01x02, TerminalBlock_Phoenix:TerminalBlock_Phoenix_MKDS-1,5-2-5.08_1x02_P5.08mm_Horizontal, B.Cu at (240.2, 136.9)
- added J7: Screw_Terminal_01x02, TerminalBlock_Phoenix:TerminalBlock_Phoenix_MKDS-1,5-2-5.08_1x02_P5.08mm_Horizontal, B.Cu at (240.2, 147.1)
- added J8: Screw_Terminal_01x02, TerminalBlock_Phoenix:TerminalBlock_Phoenix_MKDS-1,5-2-5.08_1x02_P5.08mm_Horizontal, B.Cu at (240.2, 170.6)
- added J9: Screw_Terminal_01x02, TerminalBlock_Phoenix:TerminalBlock_Phoenix_MKDS-1,5-2-5.08_1x02_P5.08mm_Horizontal, F.Cu at (183.1, 93.2)
- added L1: 2.2 μH, Inductor_SMD:L_Coilcraft_XxL4020, F.Cu at (119.7, 116.0)
- added R1: 18.2 kΩ, Resistor_SMD:R_0603_1608Metric_Pad0.98x0.95mm_HandSolder, F.Cu at (115.5, 105.8)
- added R3: 182 kΩ, Resistor_SMD:R_0603_1608Metric_Pad0.98x0.95mm_HandSolder, F.Cu at (119.8, 105.8)
- added R4: 1 MΩ, Resistor_SMD:R_0603_1608Metric_Pad0.98x0.95mm_HandSolder, F.Cu at (127.6, 105.8)
- added U2: LT8609SEV-TRPBF, LT8609SEV_TRPBF:05-08-1516_ADI, F.Cu at (121.1, 110.9)
- U1: renamed from ESP32_NodeMCU1; value ~ -> ESP32_NodeMCU1
- moved U1 25.4 mm to (210.0, 160.4)
- turned A1 to -90 degrees
Connections:
- A1 pad 1: unconnected-(A1-VIN-Pad1) -> +5V
- A1 pad 4: /IMU_SCLK -> Net-(A1-SCL_SCK)
- A1 pad 5: /IMU_MOSI -> Net-(A1-SDA_SDI)
- A1 pad 6: /IMU_MISO -> Net-(A1-DO_SDO)
- A1 pad 7: /IMU_CS -> Net-(A1-CS)
- A1 pad 8: /IMU_INT1 -> Net-(A1-INT1)
- A1 pad 9: /IMU_INT2 -> Net-(A1-INT2)
- U1 pad 1: unconnected-(ESP32_NodeMCU1-3V3-Pad1) -> +3V3
- U1 pad 10: unconnected-(ESP32_NodeMCU1-GPIO26/DAC2-Pad10) -> Net-(A2-TX)
- U1 pad 11: /IMU_CS -> Net-(A1-INT2)
- U1 pad 12: unconnected-(ESP32_NodeMCU1-GPIO14-Pad12) -> Net-(DS1-CLK)
- U1 pad 15: unconnected-(ESP32_NodeMCU1-GPIO13-Pad15) -> Net-(DS1-DIN)
- U1 pad 19: unconnected-(ESP32_NodeMCU1-Vin5V-Pad19) -> +5V
- U1 pad 27: unconnected-(ESP32_NodeMCU1-GPIO16/RX2-Pad27) -> Net-(A3-TX)
- U1 pad 28: unconnected-(ESP32_NodeMCU1-GPIO17/TX2-Pad28) -> Net-(A3-RX)
- U1 pad 30: /IMU_SCLK -> Net-(A1-SDA_SDI)
- U1 pad 31: /IMU_MISO -> Net-(A1-CS)
- U1 pad 33: unconnected-(ESP32_NodeMCU1-GPIO21/SDA-Pad33) -> Net-(DS1-DC)
- U1 pad 36: unconnected-(ESP32_NodeMCU1-GPIO22/SCL-Pad36) -> Net-(DS1-~{RST})
- U1 pad 37: /IMU_MOSI -> Net-(A1-INT1)
- U1 pad 5: /IMU_INT1 -> Net-(A1-SCL_SCK)
- U1 pad 6: /IMU_INT2 -> Net-(A1-DO_SDO)
- U1 pad 7: unconnected-(ESP32_NodeMCU1-GPIO32/ADC4-Pad7) -> Net-(A2-RX)
- U1 pad 9: unconnected-(ESP32_NodeMCU1-GPIO25/DAC1-Pad9) -> Net-(DS1-~{CS})
Other:
- board size 104.1 x 132.1 mm -> 127 x 101.6 mm
- copper layers 2 -> 4

Commit message: Electrical Update
Parts:
- removed DS1: Waveshare_2inch_LCD_ST7789VW, Waveshare_2inch_LCD_ST7789VW:Waveshare_2inch_LCD_ST7789VW
- removed the J1 at (252.7, 126.8)
- removed the J2 at (252.7, 136.9)
- removed the J3 at (252.7, 147.1)
- removed the J4 at (252.7, 157.2)
- added J10: Actuator4_CAN, Connector_PinHeader_2.54mm:PinHeader_1x02_P2.54mm_Vertical, F.Cu at (165.0, 117.2)
- added J12: Conn_01x19_Pin, Connector_PinHeader_2.54mm:PinHeader_1x19_P2.54mm_Vertical, B.Cu at (224.0, 183.3)
- added J6: Waveshare_2inch_LCD_ST7789VW, Connector_JST:JST_PH_B8B-PH-K_1x08_P2.00mm_Vertical, F.Cu at (231.4, 128.0)
- added J7: Actuator1_CAN, Connector_PinHeader_2.54mm:PinHeader_1x02_P2.54mm_Vertical, F.Cu at (255.0, 96.9)
- added J8: Actuator2_CAN, Connector_PinHeader_2.54mm:PinHeader_1x02_P2.54mm_Vertical, F.Cu at (255.0, 152.8)
- J1: renamed from J10; value Screw_Terminal_01x02 -> VBAT_INPUT; footprint TerminalBlock_Phoenix:TerminalBlock_Phoenix_MKDS-1,5-2-5.08_1x02_P5.08mm_Horizontal -> Connector_AMASS:AMASS_XT60PW-M_1x02_P7.20mm_Horizontal
- J11: value Screw_Terminal_01x02 -> Conn_01x19_Pin; footprint TerminalBlock_Phoenix:TerminalBlock_Phoenix_MKDS-1,5-2-5.08_1x02_P5.08mm_Horizontal -> Connector_PinHeader_2.54mm:PinHeader_1x19_P2.54mm_Vertical; moved to B.Cu
- J2: renamed from J5; value Screw_Terminal_01x02 -> Actuator1; moved to F.Cu
- J3: renamed from J6; value Screw_Terminal_01x02 -> Actuator2; moved to F.Cu
- J4: renamed from J7; value Screw_Terminal_01x02 -> Actuator3; moved to F.Cu
- J5: renamed from J8; value Screw_Terminal_01x02 -> Actuator4; moved to F.Cu
- J9: value Screw_Terminal_01x02 -> Actuator3_CAN; footprint TerminalBlock_Phoenix:TerminalBlock_Phoenix_MKDS-1,5-2-5.08_1x02_P5.08mm_Horizontal -> Connector_PinHeader_2.54mm:PinHeader_1x02_P2.54mm_Vertical
- moved J5 100.1 mm to (165.0, 104.5), turned to -90 degrees
- moved J11 99.3 mm to (196.0, 183.3)
- moved H1 96.0 mm to (255.0, 90.0)
- moved H2 96.0 mm to (165.0, 90.0)
- moved C1 90.1 mm to (214.7, 99.5)
- moved U1 90.1 mm to (210.1, 97.1)
- moved C2 90.1 mm to (205.0, 96.9)
- moved R2 90.1 mm to (208.9, 92.0)
- moved C3 90.1 mm to (210.6, 92.0)
- moved C4 90.1 mm to (203.8, 100.6)
- moved L1 90.1 mm to (208.7, 102.2)
- moved R1 90.1 mm to (204.5, 92.0)
- moved R3 90.0 mm to (216.6, 92.5)
- moved J9 81.9 mm to (165.0, 173.1), turned to 180 degrees
- moved J4 76.4 mm to (165.0, 160.5), turned to -90 degrees
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- renumbered C_IN1 to C1, C_VCC1 to C2, C4 to C3, C5 to C4, R3 to R2, R4 to R3, U2 to U1, U1 to U2
Connections:
- A1 pad 4: Net-(A1-SCL_SCK) -> /GPIO18
- A1 pad 5: Net-(A1-SDA_SDI) -> /GPIO23
- A1 pad 6: Net-(A1-DO_SDO) -> /GPIO19
- A1 pad 7: Net-(A1-CS) -> /GPIO27
- A1 pad 8: Net-(A1-INT1) -> /GPIO34
- A1 pad 9: Net-(A1-INT2) -> /GPIO35
- J11 pad 1: GND -> +3V3
- J11 pad 2: VBAT -> /EN
- J9 pad 1: Net-(DS1-DC) -> Net-(A2-CANH)
- J9 pad 2: Net-(DS1-~{RST}) -> Net-(A2-CANL)
- U1 pad 11: /EN -> VBAT
- U1 pad 17: unconnected-(U2-GND-Pad17) -> GND
- U2 pad 10: Net-(A2-TX) -> /GPIO26
- U2 pad 11: Net-(A1-INT2) -> /GPIO27
- U2 pad 12: Net-(DS1-CLK) -> /GPIO14
- U2 pad 13: unconnected-(U1-GPIO12-Pad13) -> /GPIO12
- U2 pad 15: Net-(DS1-DIN) -> /GPIO13
- U2 pad 16: unconnected-(U1-(RX1/F-D2)-Pad16) -> /GPIO9
- U2 pad 17: unconnected-(U1-(TX1/F-D3)-Pad17) -> /GPIO10
- U2 pad 18: unconnected-(U1-(F-CMD)-Pad18) -> /GPIO11
- U2 pad 2: unconnected-(U1-~{RST/EN}-Pad2) -> /EN
- U2 pad 20: unconnected-(U1-(F-CK)-Pad20) -> /GPIO6
- U2 pad 21: unconnected-(U1-(F-D0)-Pad21) -> /GPIO7
- U2 pad 22: unconnected-(U1-(F-D1)-Pad22) -> /GPIO8
- U2 pad 23: unconnected-(U1-GPIO15-Pad23) -> /GPIO15
- U2 pad 24: unconnected-(U1-GPIO2-Pad24) -> /GPIO2
- U2 pad 25: unconnected-(U1-GPIO0/~{PROG}-Pad25) -> /GPIO0
- U2 pad 26: unconnected-(U1-GPIO4-Pad26) -> /GPIO4
- U2 pad 27: Net-(A3-TX) -> /GPIO16
- U2 pad 28: Net-(A3-RX) -> /GPIO17
- U2 pad 29: unconnected-(U1-GPIO5-Pad29) -> /GPIO5
- U2 pad 3: unconnected-(U1-GPIO36/ADC0-Pad3) -> /GPIO36
- U2 pad 30: Net-(A1-SDA_SDI) -> /GPIO18
- U2 pad 31: Net-(A1-CS) -> /GPIO19
- U2 pad 33: Net-(DS1-DC) -> /GPIO21
- U2 pad 34: unconnected-(U1-GPIO3/RX0-Pad34) -> /GPIO3
- U2 pad 35: unconnected-(U1-GPIO1/TX0-Pad35) -> /GPIO1
- U2 pad 36: Net-(DS1-~{RST}) -> /GPIO22
- U2 pad 37: Net-(A1-INT1) -> /GPIO23
- U2 pad 4: unconnected-(U1-GPI39/ADC3-Pad4) -> /GPIO39
- U2 pad 5: Net-(A1-SCL_SCK) -> /GPIO34
- U2 pad 6: Net-(A1-DO_SDO) -> /GPIO35
- U2 pad 7: Net-(A2-RX) -> /GPIO32
- U2 pad 8: unconnected-(U1-GPIO33/ADC5-Pad8) -> /GPIO33
- U2 pad 9: Net-(DS1-~{CS}) -> /GPIO25
Routing:
- net Net-(A2-CANH): track 0.00 -> 210.0 mm, vias 0 -> 4
- net Net-(A2-CANL): track 0.00 -> 207.1 mm, vias 0 -> 2
- net VBAT: track 0.00 -> 206.3 mm
- net +5V: track 0.00 -> 165.5 mm, vias 0 -> 4
- net /GPIO23: track 0.00 -> 59.3 mm, vias 0 -> 2
- net /GPIO25: track 0.00 -> 50.1 mm, vias 0 -> 3
- net /GPIO34: track 0.00 -> 48.6 mm
- net /GPIO14: track 0.00 -> 47.4 mm, vias 0 -> 3
- net /GPIO19: track 0.00 -> 45.2 mm
- net /GPIO35: track 0.00 -> 45.0 mm
- net /GPIO13: track 0.00 -> 44.8 mm, vias 0 -> 3
- net /GPIO22: track 0.00 -> 43.8 mm
- net /GPIO18: track 0.00 -> 40.5 mm
- net /GPIO21: track 0.00 -> 38.2 mm
- net /GPIO32: track 0.00 -> 35.0 mm
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- added copper zone on B.Cu, net GND
Other:
- board size 127 x 101.6 mm -> 100 x 100 mm
- copper layers 4 -> 2

Commit message: Electrical_Save
Parts:
- J1: footprint Connector_AMASS:AMASS_XT60PW-M_1x02_P7.20mm_Horizontal -> 12GaugePower:12GaugePower
- J6: renamed from J11; value Conn_01x19_Pin -> ESP32_NodeMCU_1
- J7: renamed from J12; value Conn_01x19_Pin -> ESP32_NodeMCU_2
- moved J1 3.67 mm to (250.6, 135.0)
- renumbered J8 to J10, J9 to J11, J10 to J12, J6 to J8, J7 to J9
Routing:
- net VBAT: track 206.3 -> 207.1 mm

Commit message: R1
Parts:
- added J1: VBAT_INPUT, 12GaugePower:12GaugePower, F.Cu at (255.0, 135.0)
- added J8: BEC, Connector_PinHeader_2.54mm:PinHeader_1x04_P2.54mm_Vertical, F.Cu at (244.3, 131.2)
- moved R1 89.0 mm to (234.7, 175.8), turned to 0 degrees
- moved C4 87.1 mm to (243.5, 178.2), turned to 180 degrees
- moved C2 86.7 mm to (239.0, 176.6), turned to 90 degrees
- moved J2 85.6 mm to (165.0, 135.0), turned to 90 degrees
- moved R2 84.8 mm to (234.7, 172.8), turned to 0 degrees
- moved C3 81.9 mm to (234.8, 170.3), turned to 180 degrees
- moved U1 80.2 mm to (239.2, 171.8), turned to 90 degrees
- moved L1 79.7 mm to (245.0, 173.1), turned to 90 degrees
- moved R3 77.5 mm to (234.7, 167.8)
- moved C1 72.5 mm to (241.4, 166.9), turned to 0 degrees
- moved J7 53.6 mm to (224.0, 137.5), turned to 180 degrees
- moved J9 53.6 mm to (196.0, 137.5), turned to 180 degrees
- moved A3 50.1 mm to (184.6, 135.0), turned to -90 degrees
- moved U2 45.7 mm to (210.0, 183.3), turned to 180 degrees
- moved A2 44.3 mm to (210.0, 99.4), turned to 0 degrees
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- renumbered J8 to J14, J9 to J15, J10 to J16, J11 to J17, J12 to J18, J1 to J2, J2 to J3, J3 to J4, J4 to J5, J5 to J6, J6 to J7, J7 to J9
Routing:
- net VBAT: track 207.1 -> 158.1 mm, vias 0 -> 9
- net /GPIO26: track 27.4 -> 71.6 mm, vias 0 -> 2
- net +5V: track 165.5 -> 207.2 mm, vias 4 -> 17
- net /GPIO23: track 59.3 -> 20.7 mm, vias 2 -> 0
- net /GPIO27: track 34.7 -> 64.9 mm, vias 1 -> 0
- net /GPIO32: track 35.0 -> 65.1 mm, vias 0 -> 2
- net /GPIO13: track 44.8 -> 72.2 mm, vias 3 -> 0
- net Net-(A2-CANL): track 207.1 -> 232.5 mm
- net Net-(A2-CANH): track 210.0 -> 232.7 mm
- net /GPIO14: track 47.4 -> 65.1 mm, vias 3 -> 0
- net /GPIO21: track 38.2 -> 55.3 mm
- net /GPIO17: track 26.7 -> 42.2 mm, vias 2 -> 0
- net /GPIO16: track 28.0 -> 42.2 mm, vias 2 -> 0
- net /GPIO35: track 45.0 -> 58.5 mm, vias 0 -> 2
- net /GPIO19: track 45.2 -> 33.8 mm, vias 0 -> 2
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- added copper zone on B.Cu, net +5V
- added copper zone on F.Cu, net +5V
- added copper zone on F.Cu, net GND
- added copper zone on B.Cu, net Net-(L1-Pad2)
- added copper zone on F.Cu, net Net-(L1-Pad2)
- added copper zone on B.Cu, net VBAT
- added copper zone on F.Cu, net VBAT
