File: 03_electrical/esp32_nodemcu/esp32_nodemcu.kicad_sch (KiCad schematic)
At the start: 13 parts, among them J1 CAN_Node_3Pin, J2 CAN_Node_3Pin, J3 CAN_Node_3Pin, J4 CAN_Node_3Pin, U1 ESP32_NodeMCU1

Commit message: KiCad save
Parts:
- added C4: 10 pF, Capacitor_SMD:C_0603_1608Metric_Pad1.08x0.95mm_HandSolder, symbol Device:C
- added C5: 22 μF, Capacitor_SMD:C_1206_3216Metric_Pad1.33x1.80mm_HandSolder, symbol Device:C
- added C_IN1: 4.7 μF, Capacitor_SMD:C_1206_3216Metric_Pad1.33x1.80mm_HandSolder, symbol Device:C
- added C_VCC1: 1 μF, Capacitor_SMD:C_0603_1608Metric_Pad1.08x0.95mm_HandSolder, symbol Device:C
- added J10, J11, J5, J6, J7, J8, J9: Screw_Terminal_01x02, TerminalBlock_Phoenix:TerminalBlock_Phoenix_MKDS-1,5-2-5.08_1x02_P5.08mm_Horizontal, symbol Connector:Screw_Terminal_01x02
- added L1: 2.2 μH, Inductor_SMD:L_Coilcraft_XxL4020, symbol Device:L
- added R1: 18.2 kΩ, Resistor_SMD:R_0603_1608Metric_Pad0.98x0.95mm_HandSolder, symbol Device:R_US
- added R3: 182 kΩ, Resistor_SMD:R_0603_1608Metric_Pad0.98x0.95mm_HandSolder, symbol Device:R_US
- added R4: 1 MΩ, Resistor_SMD:R_0603_1608Metric_Pad0.98x0.95mm_HandSolder, symbol Device:R_US
- added U2: LT8609SEV-TRPBF, LT8609SEV_TRPBF:05-08-1516_ADI, symbol LT8609SEV_TRPBF:LT8609SEV-TRPBF
- H1, H2, H3, H4: footprint (none) -> MountingHole:MountingHole_3.5mm_Pad_TopBottom
- J1, J2, J3, J4: footprint (none) -> Connector_PinHeader_2.54mm:PinHeader_1x03_P2.54mm_Vertical
Connections:
- net GND: now also C5.2, C_IN1.2, C_VCC1.1, J10.1 (Pin_1), J11.1 (Pin_1), J5.1 (Pin_1), J6.1 (Pin_1), J7.1 (Pin_1), J8.1 (Pin_1), R1.1, R3.1, U2.14 (GND), U2.3 (GND), U2.4 (GND), U2.8 (GND)
- net +5V: now reaches A2.1 (VCC)
- net +5V: now also A1.1 (VIN), A3.3 (5V), DS1.1 (VCC), U1.19 (Vin5V), C4.2, C5.1, L1.1, R4.1
- net at A2.3 (RX): now also U1.7 (GPIO32/ADC4)
- net at A2.4 (TX): now also U1.10 (GPIO26/DAC2)
- net at DS1.3 (DIN): now also U1.15 (GPIO13)
- net at DS1.4 (CLK): now also U1.12 (GPIO14)
- net at DS1.5 (~{CS}): now also U1.9 (GPIO25/DAC1)
- net at DS1.6 (DC): now also U1.33 (GPIO21/SDA), J9.1 (Pin_1)
- net at DS1.7 (~{RST}): now also U1.36 (GPIO22/SCL), J9.2 (Pin_2)
- net +3V3: now reaches DS1.8 (BL)
- net +3V3: now also U1.1 (3V3)
- net at A3.1 (RX): now also U1.28 (GPIO17/TX2)
- net at A3.2 (TX): now also U1.27 (GPIO16/RX2)
- net IMU_CS: no longer names the net of U1.11 (GPIO27)
- net IMU_CS: now also A1.9 (INT2); no longer A1.7 (CS)
- net IMU_INT1: no longer names the net of A1.8 (INT1)
- net IMU_INT1: now also U1.37 (GPIO23/COPI); no longer U1.5 (GPI34/ADC6)
- net IMU_INT2: no longer names the net of U1.6 (GPI35/ADC7)
- net IMU_INT2: now also A1.6 (DO_SDO); no longer A1.9 (INT2)
- net IMU_MISO: no longer names the net of U1.31 (GPIO19/CIPO)
- net IMU_MISO: now also A1.7 (CS); no longer A1.6 (DO_SDO)
- net IMU_MOSI: no longer names the net of A1.5 (SDA_SDI)
- net IMU_MOSI: now also U1.30 (GPIO18/SCK); no longer U1.37 (GPIO23/COPI)
- net IMU_SCLK: no longer names the net of A1.4 (SCL_SCK)
- net IMU_SCLK: now also U1.5 (GPI34/ADC6); no longer U1.30 (GPIO18/SCK)
- new net: C4.1, R3.2, R4.2, U2.13 (FB)
- new net: C_VCC1.2, U2.2 (VCC)
- new net: L1.2, U2.5 (SW), U2.6 (SW)
- new net: R1.2, U2.1 (RT)
- new net EN: U2.11 (EN/UV)
- new net VBAT: C_IN1.1, J10.2 (Pin_2), J11.2 (Pin_2), J5.2 (Pin_2), J6.2 (Pin_2), J7.2 (Pin_2), J8.2 (Pin_2), U2.10 (VIN), U2.9 (VIN)
- no-connect marks 0 -> 27
Other:
- removed sheet Power
- note added: "I2C_SCL"
- note added: "I2C_SDA"
- moved on the sheet: H1, H2, H3, H4

Commit message: Electrical Update
Parts:
- removed DS1: Waveshare_2inch_LCD_ST7789VW, Waveshare_2inch_LCD_ST7789VW:Waveshare_2inch_LCD_ST7789VW, symbol Waveshare_2inch_LCD_ST7789VW:Waveshare_2inch_LCD_ST7789VW
- removed J1, J2, J3, J4: CAN_Node_3Pin, Connector_PinHeader_2.54mm:PinHeader_1x03_P2.54mm_Vertical, symbol CAN_Node_3Pin:CAN_Node_3Pin
- removed J11, J9: Screw_Terminal_01x02, TerminalBlock_Phoenix:TerminalBlock_Phoenix_MKDS-1,5-2-5.08_1x02_P5.08mm_Horizontal, symbol Connector:Screw_Terminal_01x02
- added J10: Actuator4_CAN, Connector_PinHeader_2.54mm:PinHeader_1x02_P2.54mm_Vertical, symbol Connector:Conn_01x02_Pin
- added J11, J12: Conn_01x19_Pin, Connector_PinHeader_2.54mm:PinHeader_1x19_P2.54mm_Vertical, symbol Connector:Conn_01x19_Pin
- added J6: Waveshare_2inch_LCD_ST7789VW, Connector_JST:JST_PH_B8B-PH-K_1x08_P2.00mm_Vertical, symbol Connector:Conn_01x08_Pin
- added J7: Actuator1_CAN, Connector_PinHeader_2.54mm:PinHeader_1x02_P2.54mm_Vertical, symbol Connector:Conn_01x02_Pin
- added J8: Actuator2_CAN, Connector_PinHeader_2.54mm:PinHeader_1x02_P2.54mm_Vertical, symbol Connector:Conn_01x02_Pin
- added J9: Actuator3_CAN, Connector_PinHeader_2.54mm:PinHeader_1x02_P2.54mm_Vertical, symbol Connector:Conn_01x02_Pin
- J1: renamed from J10; value Screw_Terminal_01x02 -> VBAT_INPUT; footprint TerminalBlock_Phoenix:TerminalBlock_Phoenix_MKDS-1,5-2-5.08_1x02_P5.08mm_Horizontal -> Connector_AMASS:AMASS_XT60PW-M_1x02_P7.20mm_Horizontal
- J2: renamed from J5; value Screw_Terminal_01x02 -> Actuator1
- J3: renamed from J6; value Screw_Terminal_01x02 -> Actuator2
- J4: renamed from J7; value Screw_Terminal_01x02 -> Actuator3
- J5: renamed from J8; value Screw_Terminal_01x02 -> Actuator4
- renumbered C_IN1 to C1, C_VCC1 to C2, C4 to C3, C5 to C4, R3 to R2, R4 to R3, U2 to U1, U1 to U2
Connections:
- net +3V3: now also J11.1 (Pin_1)
- net +5V: now also J11.19 (Pin_19), J6.1 (Pin_1), J6.8 (Pin_8)
- net EN: now also U2.2 (~{RST/EN}), J11.2 (Pin_2); no longer U1.11 (EN/UV)
- net GND: now also U1.17 (GND), J11.14 (Pin_14), J12.1 (Pin_1), J12.7 (Pin_7), J6.2 (Pin_2)
- net VBAT: now also U1.11 (EN/UV)
- net at A2.6 (CANH): now also J10.1 (Pin_1), J7.1 (Pin_1), J8.1 (Pin_1), J9.1 (Pin_1)
- net at A2.7 (CANL): now also J10.2 (Pin_2), J7.2 (Pin_2), J8.2 (Pin_2), J9.2 (Pin_2)
- net GPIO32: now reaches A2.3 (RX), U2.7 (GPIO32/ADC4)
- net GPIO32: now also J11.7 (Pin_7)
- net GPIO26: now reaches A2.4 (TX), U2.10 (GPIO26/DAC2)
- net GPIO26: now also J11.10 (Pin_10)
- net GPIO13: now reaches U2.15 (GPIO13)
- net GPIO13: now also J11.15 (Pin_15), J6.3 (Pin_3)
- net GPIO14: now reaches U2.12 (GPIO14)
- net GPIO14: now also J11.12 (Pin_12), J6.4 (Pin_4)
- net GPIO25: now reaches U2.9 (GPIO25/DAC1)
- net GPIO25: now also J11.9 (Pin_9), J6.5 (Pin_5)
- net GPIO21: now reaches U2.33 (GPIO21/SDA)
- net GPIO21: now also J12.6 (Pin_6), J6.6 (Pin_6)
- net GPIO22: now reaches U2.36 (GPIO22/SCL)
- net GPIO22: now also J12.3 (Pin_3), J6.7 (Pin_7)
- net GPIO17: now reaches A3.1 (RX), U2.28 (GPIO17/TX2)
- net GPIO17: now also J12.11 (Pin_11)
- net GPIO16: now reaches A3.2 (TX), U2.27 (GPIO16/RX2)
- net GPIO16: now also J12.12 (Pin_12)
- net GPIO27: now reaches U2.11 (GPIO27)
- net GPIO27: now also A1.7 (CS), J11.11 (Pin_11); no longer A1.9 (INT2)
- net GPIO12: now reaches U2.13 (GPIO12)
- net GPIO12: now also J11.13 (Pin_13)
- net GPIO9: now reaches U2.16 ((RX1/F-D2))
- net GPIO9: now also J11.16 (Pin_16)
- net GPIO10: now reaches U2.17 ((TX1/F-D3))
- net GPIO10: now also J11.17 (Pin_17)
- net GPIO11: now reaches U2.18 ((F-CMD))
- net GPIO11: now also J11.18 (Pin_18)
- net GPIO6: now reaches U2.20 ((F-CK))
- net GPIO6: now also J12.19 (Pin_19)
- net GPIO7: now reaches U2.21 ((F-D0))
- net GPIO7: now also J12.18 (Pin_18)
- net GPIO8: now reaches U2.22 ((F-D1))
- net GPIO8: now also J12.17 (Pin_17)
- net GPIO15: now reaches U2.23 (GPIO15)
- net GPIO15: now also J12.16 (Pin_16)
- net GPIO2: now reaches U2.24 (GPIO2)
- net GPIO2: now also J12.15 (Pin_15)
- net GPIO0: now reaches U2.25 (GPIO0/~{PROG})
- net GPIO0: now also J12.14 (Pin_14)
- net GPIO4: now reaches U2.26 (GPIO4)
- net GPIO4: now also J12.13 (Pin_13)
- net GPIO5: now reaches U2.29 (GPIO5)
- net GPIO5: now also J12.10 (Pin_10)
- net GPIO36: now reaches U2.3 (GPIO36/ADC0)
- net GPIO36: now also J11.3 (Pin_3)
- net GPIO18: now reaches U2.30 (GPIO18/SCK)
- net GPIO18: now also A1.4 (SCL_SCK), J12.9 (Pin_9); no longer A1.5 (SDA_SDI)
- net GPIO19: now reaches U2.31 (GPIO19/CIPO)
- net GPIO19: now also A1.6 (DO_SDO), J12.8 (Pin_8); no longer A1.7 (CS)
- net GPIO3: now reaches U2.34 (GPIO3/RX0)
- net GPIO3: now also J12.5 (Pin_5)
- net GPIO1: now reaches U2.35 (GPIO1/TX0)
- net GPIO1: now also J12.4 (Pin_4)
- net GPIO23: now reaches U2.37 (GPIO23/COPI)
- net GPIO23: now also A1.5 (SDA_SDI), J12.2 (Pin_2); no longer A1.8 (INT1)
- net GPIO39: now reaches U2.4 (GPI39/ADC3)
- net GPIO39: now also J11.4 (Pin_4)
- net GPIO34: now reaches U2.5 (GPI34/ADC6)
- net GPIO34: now also A1.8 (INT1), J11.5 (Pin_5); no longer A1.4 (SCL_SCK)
- net GPIO35: now reaches U2.6 (GPI35/ADC7)
- net GPIO35: now also A1.9 (INT2), J11.6 (Pin_6); no longer A1.6 (DO_SDO)
- net GPIO33: now reaches U2.8 (GPIO33/ADC5)
- net GPIO33: now also J11.8 (Pin_8)
Other:
- note added: "CANH CANL"
- note added: "VCC GND DIN CLK CS DS RST BL"
- note removed: "I2C_SCL"
- note removed: "I2C_SDA"
- moved on the sheet: C1, C2, C3, C4, H1, H2, H3, H4, J1, J2, J3, J4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

Commit message: Electrical_Save
Parts:
- removed J1: VBAT_INPUT, Connector_AMASS:AMASS_XT60PW-M_1x02_P7.20mm_Horizontal, symbol Connector:Screw_Terminal_01x02
- added J1: VBAT_INPUT, 12GaugePower:12GaugePower, symbol Connector:Conn_01x02_Pin
- J6: renamed from J11; value Conn_01x19_Pin -> ESP32_NodeMCU_1
- J7: renamed from J12; value Conn_01x19_Pin -> ESP32_NodeMCU_2
- U1: footprint LT8609SEV_TRPBF:05-08-1516_ADI -> 05-08-1516_ADI
- renumbered J8 to J10, J9 to J11, J10 to J12, J6 to J8, J7 to J9
Connections:
- net GND: now also J1.1 (Pin_1)
- net VBAT: now also J1.2 (Pin_2)

Commit message: R1
Parts:
- added J1: VBAT_INPUT, 12GaugePower:12GaugePower, symbol Connector:Conn_01x02_Pin
- added J8: BEC, Connector_PinHeader_2.54mm:PinHeader_1x04_P2.54mm_Vertical, symbol Connector:Conn_01x04_Pin
- U1: footprint 05-08-1516_ADI -> LT8609SEV_TRPBF:05-08-1516_ADI
- renumbered J8 to J14, J9 to J15, J10 to J16, J11 to J17, J12 to J18, J1 to J2, J2 to J3, J3 to J4, J4 to J5, J5 to J6, J6 to J7, J7 to J9
Connections:
- net +5V: now also J8.4 (Pin_4)
- net GND: now also J1.1 (Pin_1), J8.2 (Pin_2), J8.3 (Pin_3)
- net VBAT: now also J1.2 (Pin_2), J8.1 (Pin_1)
Other:
- moved on the sheet: J2, J3, J4, J5, J6
